File: hw/pcb/mp3Player/power.kicad_sch (KiCad schematic)
At the start: 0 parts

Commit message: updates to pcb to supported updated rtl
Parts:
- added C7, C8: C_Polarized, symbol Device:C_Polarized
- added R1, R7: R, symbol Device:R
- added U3: LM317_TO-220, Package_TO_SOT_THT:TO-220-3_Vertical, symbol Regulator_Linear:LM317_TO-220
Connections:
- new net: R1.2, R7.1, U3.1 (ADJ)
- new net +3.3V: C8.1, R1.1, U3.2 (VO)
- new net +5V: C7.1, U3.3 (VI)
- new net GND: C7.2, C8.2, R7.2
